File: Pcb timer analogique v0/Detection.kicad_sch (KiCad schematic)
At the start: 0 parts

Commit message: Partie detection du timer analaogique
Parts:
- added C1: 1.6u, symbol Device:C_Small
- added C2: 100n, symbol Device:C_Small
- added R1, R2, R5: 10k, symbol Device:R_Small
- added R3: 5.6k, symbol Device:R_Small
- added R4: 1M, symbol Device:R_Small
- added U2: ADXL335BCPZ, ADXL335BCPZ:PQFN65P400X400X150-17N, symbol ADXL335BCPZ:ADXL335BCPZ
- added U3: LM393, symbol Comparator:LM393
Connections:
- new net: R4.2, R5.1, U3.1
- new net: U2.1 (NC), U2.11 (NC), U2.13 (NC), U2.16 (NC), U2.4 (NC), U2.9 (NC)
- new net: R1.1, U2.10 (YOUT)
- new net +3.3V: C2.2, U2.14 (VS), U2.15 (VS)
- new net +5V: R2.1, R5.2
- new net COM: C1.2, C2.1, R3.2, U2.2 (ST), U2.3 (COM), U2.5 (COM), U2.6 (COM), U2.7 (COM), U3.5 (+), U3.6 (-)
- new net V_filtree: C1.1, R1.2, U3.2 (-)
- new net Vref: R2.2, R3.1, R4.1, U3.3 (+)
- no-connect marks 0 -> 5
Other:
- note added: "Hystéresis"
- note added: "Pont diviseur de tension qui délivre du 5V"
- note added: "Résistance pull up"
